File: Lab4/lab4exercise1/lab4.kicad_sch (KiCad schematic)
At the start: 6 parts, among them SW1 SW_SPDT

Commit message: finished
Other:
- title: (none) -> Lab 4 Exercise 1
Changed lines of the file:
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@@
 (kicad_sch (version 20211123) (generator eeschema)
   (paper "A4")
+  (title_block
+    (title "Lab 4 Exercise 1")
+  )
   (junction (at 217.17 115.57) (diameter 0) (color 0 0 0 0)
   )

Commit message: finished pcb schematic
Parts:
- C1: footprint (none) -> Capacitor_THT:CP_Radial_D5.0mm_P2.00mm
- D1: footprint (none) -> LED_THT:LED_D5.0mm
- R1, R2: footprint (none) -> Resistor_THT:R_Axial_DIN0516_L15.5mm_D5.0mm_P20.32mm_Horizontal
- SW1: footprint (none) -> Button_Switch_THT:SW_E-Switch_EG1224_SPDT_Angled
- V1: footprint (none) -> Connector_JST:JST_PH_B2B-PH-K_1x02_P2.00mm_Vertical
Connections:
- net GND: no longer names the net of C1.2, D1.1 (K), V1.2 (Pin_2)
Changed lines of the file:
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@@
     (title "Lab 4 Exercise 1")
   )
-  (junction (at 217.17 115.57) (diameter 0) (color 0 0 0 0)
+  (junction (at 190.5 115.57) (diameter 0) (color 0 0 0 0)
   )
   (junction (at 190.5 99.06) (diameter 0) (color 0 0 0 0)
   )
-  (junction (at 190.5 115.57) (diameter 0) (color 0 0 0 0)
-  )
   (wire (pts (xy 151.13 96.52) (xy 153.67 96.52))
-    (stroke (width 0) (type default) (color 0 0 0 0))
-  )
-  (wire (pts (xy 217.17 115.57) (xy 217.17 116.84))
     (stroke (width 0) (type default) (color 0 0 0 0))
   )
@@
     (stroke (width 0) (type default) (color 0 0 0 0))
   )
+  (wire (pts (xy 190.5 115.57) (xy 217.17 115.57))
+    (stroke (width 0) (type default) (color 0 0 0 0))
+  )
   (wire (pts (xy 217.17 106.68) (xy 217.17 107.95))
     (stroke (width 0) (type default) (color 0 0 0 0))
   )
   (wire (pts (xy 190.5 115.57) (xy 151.13 115.57))
-    (stroke (width 0) (type default) (color 0 0 0 0))
-  )
-  (wire (pts (xy 217.17 115.57) (xy 190.5 115.57))
     (stroke (width 0) (type default) (color 0 0 0 0))
   )
@@
       (effects (font (size 1.27 1.27)) (justify right))
     )
-    (property "Footprint" "" (id 2) (at 217.17 111.76 0)
+    (property "Footprint" "LED_THT:LED_D5.0mm" (id 2) (at 217.17 111.76 0)
       (effects (font (size 1.27 1.27)) hide)
     )
@@
     (property "Reference" "V1" (id 0) (at 146.685 99.06 0))
     (property "Value" "9V" (id 1) (at 146.685 101.6 0))
-    (property "Footprint" "" (id 2) (at 146.05 104.14 0)
+    (property "Footprint" "Connector_JST:JST_PH_B2B-PH-K_1x02_P2.00mm_Vertical" (id 2) (at 146.05 104.14 0)
       (effects (font (size 1.27 1.27)) hide)
     )
@@
     (pin "2")
   )
-  (symbol (lib_id "power:GND") (at 217.17 116.84 0) (unit 1)
-    (in_bom yes) (on_board yes) (fields_autoplaced)
-    (property "Reference" "#PWR?" (id 0) (at 217.17 123.19 0)
-      (effects (font (size 1.27 1.27)) hide)
-    )
-    (property "Value" "GND" (id 1) (at 217.17 121.92 0))
-    (property "Footprint" "" (id 2) (at 217.17 116.84 0)
-      (effects (font (size 1.27 1.27)) hide)
-    )
-    (property "Datasheet" "" (id 3) (at 217.17 116.84 0)
-      (effects (font (size 1.27 1.27)) hide)
-    )
-    (pin "1")
-  )
   (symbol (lib_id "Switch:SW_SPDT") (at 173.99 96.52 0) (unit 1)
     (in_bom yes) (on_board yes) (fields_autoplaced)
@@
       (effects (font (size 1.27 1.27)) hide)
     )
-    (property "Footprint" "" (id 2) (at 173.99 96.52 0)
+    (property "Footprint" "Button_Switch_THT:SW_E-Switch_EG1224_SPDT_Angled" (id 2) (at 173.99 96.52 0)
       (effects (font (size 1.27 1.27)) hide)
     )
@@
     (property "Reference" "R2" (id 0) (at 157.48 90.17 90))
     (property "Value" "2.2kR" (id 1) (at 157.48 92.71 90))
-    (property "Footprint" "" (id 2) (at 157.48 94.742 90)
+    (property "Footprint" "Resistor_THT:R_Axial_DIN0516_L15.5mm_D5.0mm_P20.32mm_Horizontal" (id 2) (at 157.48 94.742 90)
       (effects (font (size 1.27 1.27)) hide)
     )
@@
       (effects (font (size 1.27 1.27)) (justify left))
     )
-    (property "Footprint" "" (id 2) (at 215.392 102.87 90)
+    (property "Footprint" "Resistor_THT:R_Axial_DIN0516_L15.5mm_D5.0mm_P20.32mm_Horizontal" (id 2) (at 215.392 102.87 90)
       (effects (font (size 1.27 1.27)) hide)
     )
@@
       (effects (font (size 1.27 1.27)) (justify left))
     )
-    (property "Footprint" "" (id 2) (at 191.4652 109.22 0)
+    (property "Footprint" "Capacitor_THT:CP_Radial_D5.0mm_P2.00mm" (id 2) (at 191.4652 109.22 0)
       (effects (font (size 1.27 1.27)) hide)
     )
@@
   )
   (symbol_instances
-    (path "/4b49338b-c922-4426-831e-54bfc0e6179c"
-      (reference "#PWR?") (unit 1) (value "GND") (footprint "")
-    )
     (path "/cccf5c5a-300a-4fcc-ace3-eade91121582"
-      (reference "C1") (unit 1) (value "4.7uF") (footprint "")
+      (reference "C1") (unit 1) (value "4.7uF") (footprint "Capacitor_THT:CP_Radial_D5.0mm_P2.00mm")
     )
     (path "/241ab488-fb00-4de4-9343-282b8f591571"
-      (reference "D1") (unit 1) (value "LED") (footprint "")
+      (reference "D1") (unit 1) (value "LED") (footprint "LED_THT:LED_D5.0mm")
     )
     (path "/b5f1c06c-689a-495d-b1b0-d525c44bf58d"
-      (reference "R1") (unit 1) (value "20kR") (footprint "")
+      (reference "R1") (unit 1) (value "20kR") (footprint "Resistor_THT:R_Axial_DIN0516_L15.5mm_D5.0mm_P20.32mm_Horizontal")
     )
     (path "/8e2a1812-e3e7-47fd-9542-415acdce6b36"
-      (reference "R2") (unit 1) (value "2.2kR") (footprint "")
+      (reference "R2") (unit 1) (value "2.2kR") (footprint "Resistor_THT:R_Axial_DIN0516_L15.5mm_D5.0mm_P20.32mm_Horizontal")
     )
     (path "/5a3be1f4-8143-4422-a8e0-28a84ffedc3a"
-      (reference "SW1") (unit 1) (value "SW_SPDT") (footprint "")
+      (reference "SW1") (unit 1) (value "SW_SPDT") (footprint "Button_Switch_THT:SW_E-Switch_EG1224_SPDT_Angled")
     )
     (path "/4ab5ce02-55ae-4e0c-a184-b7c68a7ecf9a"
-      (reference "V1") (unit 1) (value "9V") (footprint "")
+      (reference "V1") (unit 1) (value "9V") (footprint "Connector_JST:JST_PH_B2B-PH-K_1x02_P2.00mm_Vertical")
     )
   )
